File: PCBs/FineMotion-5.kicad_sch (KiCad schematic)
At the start: 40 parts, among them J1 Conn_01x02_Female, J2 Conn_01x04_Female, P1 USB_C_Plug_USB2.0, SW1 Option/FLASH Switch, SW3 SW_SPDT MAIN POWER, U1 ME6211C, U2 TP4056, U6 ESP-12F, U7 CH340C, U9 MPU-9250

Commit message: Update PCB Remark
Other:
- company: github.com/Kamilake/KTracker-SlimeVR-PCB -> https://github.com/Kamilake/FineMotion-Tracker
- moved on the sheet: C13
